File: PortSide.kicad_sch (KiCad schematic)
At the start: 32 parts, among them J1 Conn_ARM_JTAG_SWD_10, J2 USB_C_Receptacle_USB2.0_14P, J3 Conn_01x14, J4 Conn_02x08_Top_Bottom, Q1 2N7002, Q2 MMDT3904, U1 TCAN3404, U2 ESP32-S3-WROOM-1, U3 AP2112K-3.3, U4 INA226, U5 LM5164DDA, U7 CP2102N-Axx-xQFN24

Commit message: Version 2, still not happy with that
Parts:
- removed J3: Conn_01x14, Connector_PinSocket_2.54mm:PinSocket_1x14_P2.54mm_Vertical, symbol Connector_Generic:Conn_01x14
- added J5: Conn_02x07_Counter_Clockwise, Connector_PinHeader_2.54mm:PinHeader_2x07_P2.54mm_Vertical, symbol Connector_Generic:Conn_02x07_Counter_Clockwise
- J1: footprint Connector_IDC:IDC-Header_2x05_P2.54mm_Vertical_SMD -> Connector_IDC:IDC-Header_2x05_P2.54mm_Vertical
- J2: footprint Connector_USB:USB_C_Receptacle_Amphenol_12401610E4-2A -> Connector_USB:USB_C_Receptacle_Amphenol_12401948E412A
Connections:
- net +3.3V: now also J5.1 (Pin_1)
- net CAN_RXD: now also U2.38 (IO2); no longer U2.31 (IO38)
- net CAN_TXD: now also U2.39 (IO1); no longer U2.30 (IO37)
- net GND: now also J5.2 (Pin_2)
- net INA226_ALERT: now also U2.19 (IO11); no longer U2.6 (IO6)
- net LCD_CS: now also U2.34 (IO41), J5.3 (Pin_3); no longer U2.15 (IO3)
- net LCD_DC: now also U2.33 (IO40), J5.5 (Pin_5); no longer U2.17 (IO9)
- net LCD_LED: now also U2.24 (IO47), J5.8 (Pin_8); no longer U2.20 (IO12)
- net LCD_MISO: now also U2.31 (IO38), J5.9 (Pin_9); no longer U2.21 (IO13)
- net LCD_MOSI: now also U2.23 (IO21), J5.6 (Pin_6); no longer U2.18 (IO10)
- net LCD_RESET: now also U2.22 (IO14), J5.4 (Pin_4); no longer U2.16 (IO46)
- net LCD_SCK: now also U2.32 (IO39), J5.7 (Pin_7); no longer U2.19 (IO11)
- net LCD_T_CLK: now also U2.25 (IO48), J5.10 (Pin_10); no longer U2.22 (IO14)
- net LCD_T_CS: now also U2.30 (IO37), J5.11 (Pin_11); no longer U2.23 (IO21)
- net LCD_T_DIN: now also U2.26 (IO45), J5.12 (Pin_12); no longer U2.24 (IO47)
- net LCD_T_DO: now also U2.29 (IO36), J5.13 (Pin_13); no longer U2.25 (IO48)
- net LCD_T_IRQ: now also U2.28 (IO35), J5.14 (Pin_14); no longer U2.26 (IO45)
- net MTCK: now also U2.5 (IO5); no longer U2.33 (IO40)
- net MTDI: now also U2.7 (IO7); no longer U2.35 (IO42)
- net MTDO: now also U2.6 (IO6); no longer U2.34 (IO41)
- net MTMS: now also U2.4 (IO4); no longer U2.32 (IO39)
- net SCL: now also R7.1, U2.17 (IO9); no longer R6.1, U2.4 (IO4)
- net SDA: now also R6.1, U2.18 (IO10); no longer R7.1, U2.5 (IO5)
- net TCAN3404_SHDN: now also U2.8 (IO15); no longer U2.28 (IO35)
- net TCAN3404_STB: now also U2.9 (IO16); no longer U2.29 (IO36)
Other:
- moved on the sheet: R6

Commit message: Rev 3, happy. Removed INA226 and JTAG
Parts:
- removed J1: Conn_ARM_JTAG_SWD_10, Connector_IDC:IDC-Header_2x05_P2.54mm_Vertical, symbol Connector:Conn_ARM_JTAG_SWD_10
- removed R1: 10m, Resistor_SMD:R_1206_3216Metric_Pad1.30x1.75mm_HandSolder, symbol Device:R
- removed R6, R7: 4.7k, Resistor_SMD:R_0603_1608Metric_Pad0.98x0.95mm_HandSolder, symbol Device:R
- removed U4: INA226, Package_SO:TSSOP-10_3x3mm_P0.5mm, symbol Sensor_Energy:INA226
- added D3: US1J, Diode_SMD:D_SMA, symbol Diode:US1J
- added R16, R17: 10k, Resistor_SMD:R_0603_1608Metric_Pad0.98x0.95mm_HandSolder, symbol Device:R
- C1, C3, R10, R11, R12, R13, R14, R15, R2, R3, R4, R5, R8, R9: KiLib_Generator (none) -> SMD_2terminal_chip_molded
- J4, J5: KiLib_Generator (none) -> connector/pin_header_socket
- Q1, Q2, U1, U3, U5: KiLib_Generator (none) -> package/gullwing
- U7: KiLib_Generator (none) -> package/no_lead
Connections:
- net +5V is gone; now on net 5v_SOURCE: U3.1 (VIN), U3.3 (EN)
- net MTCK is gone; now on net CAN_TXD: U2.5 (IO5)
- net MTDO is gone; now on net CAN_RXD: U2.6 (IO6)
- net CAN_RXD: no longer U2.38 (IO2)
- net CAN_TXD: no longer U2.39 (IO1)
- net CAR_POS: now also D3.1 (K); no longer J4.16 (Pin_16)
- net ESP_EN: now also R17.2
- net ESP_IO0: now also R16.1
- net GND: now also R16.2, R17.1
- net LCD_CS: now also U2.35 (IO42); no longer U2.34 (IO41)
- net LCD_DC: now also U2.34 (IO41); no longer U2.33 (IO40)
- net LCD_LED: now also U2.25 (IO48); no longer U2.24 (IO47)
- net LCD_MISO: now also U2.32 (IO39); no longer U2.31 (IO38)
- net LCD_MOSI: now also U2.39 (IO1); no longer U2.23 (IO21)
- net LCD_RESET: now also U2.38 (IO2); no longer U2.22 (IO14)
- net LCD_SCK: now also U2.33 (IO40); no longer U2.32 (IO39)
- net LCD_T_CLK: now also U2.26 (IO45); no longer U2.25 (IO48)
- net LCD_T_CS: now also U2.31 (IO38); no longer U2.30 (IO37)
- net LCD_T_DIN: now also U2.28 (IO35); no longer U2.26 (IO45)
- net LCD_T_DO: now also U2.30 (IO37); no longer U2.29 (IO36)
- net LCD_T_IRQ: now also U2.29 (IO36); no longer U2.28 (IO35)
- net TCAN3404_SHDN: now also U2.9 (IO16); no longer U2.8 (IO15)
- net TCAN3404_STB: now also U2.8 (IO15); no longer U2.9 (IO16)
- net INA226_ALERT: no longer names the net of U2.19 (IO11)
- net MTDI: no longer names the net of U2.7 (IO7)
- net MTMS: no longer names the net of U2.4 (IO4)
- net SCL: no longer names the net of U2.17 (IO9)
- net SDA: no longer names the net of U2.18 (IO10)
- new net: D3.2 (A), J4.16 (Pin_16)
Other:
- note removed: "Remember to blow fuses for this!"
- moved on the sheet: Q2A, Q2B, R8, R9
