File: Circuits/ESP32_programmer/ESP32_programmer.kicad_sch (KiCad schematic)
At the start: 0 parts

Commit message: Programmer board done??
Parts:
- added C1, C4: 4.7uF, Capacitor_SMD:C_0805_2012Metric_Pad1.18x1.45mm_HandSolder, symbol Device:C
- added C2, C3: 0.1uF, Capacitor_SMD:C_0805_2012Metric_Pad1.18x1.45mm_HandSolder, symbol Device:C
- added H1, H2, H3, H4: MountingHole_Pad, MountingHole:MountingHole_2.7mm_M2.5_ISO14580_Pad, symbol Mechanical:MountingHole_Pad
- added J1: Conn_01x06_Pin, Connector_PinSocket_2.54mm:PinSocket_1x06_P2.54mm_Vertical, symbol Connector:Conn_01x06_Pin
- added J2: USB_C_Receptacle_USB2.0_14P, Connector_USB:USB_C_Receptacle_Amphenol_12401948E412A, symbol Connector:USB_C_Receptacle_USB2.0_14P
- added Q2: MMDT3904, Package_TO_SOT_SMD:SOT-363_SC-70-6, symbol Transistor_BJT:MMDT3904
- added R1, R2: 5.1k, Resistor_SMD:R_0603_1608Metric_Pad0.98x0.95mm_HandSolder, symbol Device:R
- added R16, R17: 10k, Resistor_SMD:R_0603_1608Metric_Pad0.98x0.95mm_HandSolder, symbol Device:R
- added R3, R4, R5: 1k, Resistor_SMD:R_0603_1608Metric_Pad0.98x0.95mm_HandSolder, symbol Device:R
- added U1: TPD4S014, Package_SON:Texas_S-PWSON-N10_ThermalVias, symbol Power_Protection:TPD4S014
- added U7: CP2102N-Axx-xQFN24, Package_DFN_QFN:QFN-24-1EP_4x4mm_P0.5mm_EP2.6x2.6mm, symbol Interface_USB:CP2102N-Axx-xQFN24
Connections:
- new net: R5.1, U7.9 (~{RST})
- new net: C3.1, C4.1, R5.2, U7.5 (VIO), U7.6 (VDD)
- new net: J2.A5 (CC1), R2.1
- new net: J2.B5 (CC2), R1.1
- new net: Q2.2 (B1), R3.2
- new net: Q2.5 (B2), R4.2
- new net DTR: Q2.1 (E1), R4.1, U7.23 (~{DTR})
- new net ESP_EN: J1.6 (Pin_6), Q2.3 (C2), R17.2
- new net ESP_IO0: J1.5 (Pin_5), Q2.6 (C1), R16.1
- new net GND: C1.2, C2.2, C3.2, C4.2, H1.1, H2.1, H3.1, H4.1, J1.2 (Pin_2), J2.A1 (GND), J2.A12 (GND), J2.B1 (GND), J2.B12 (GND), J2.SH (SHIELD), R1.2, R16.2, R17.1, R2.2, U1.11 (PAD), U1.3 (~{EN}), U1.8 (GND), U7.2 (GND), U7.25 (GND)
- new net RTS: Q2.4 (E2), R3.1, U7.19 (~{RTS})
- new net RX: J1.4 (Pin_4), U7.20 (RXD)
- new net TX: J1.3 (Pin_3), U7.21 (TXD)
- new net USB+: J2.A6 (D+), J2.B6 (D+), U1.7 (D+), U7.3 (D+)
- new net USB-: J2.A7 (D-), J2.B7 (D-), U1.6 (D-), U7.4 (D-)
- new net USB_VBUS: J2.A4 (VBUS), J2.A9 (VBUS), J2.B4 (VBUS), J2.B9 (VBUS), U1.10 (VBUS), U1.9 (VBUS)
- new net VCC: C1.1, C2.1, J1.1 (Pin_1), U1.1 (VBUSOUT), U1.2 (VBUSOUT), U7.7 (VREGIN), U7.8 (VBUS)
- no-connect marks 0 -> 12
Other:
- note added: "Figure 2.6 of datasheet Self-powered devices should have this divider from VBUS to protect it from something"

Commit message: Full redesign of connector board, including removal of USB flashing. This is now done by the flasher board.
Parts:
- removed H1, H2, H3, H4: MountingHole_Pad, MountingHole:MountingHole_2.7mm_M2.5_ISO14580_Pad, symbol Mechanical:MountingHole_Pad
- removed R16, R17: 10k, Resistor_SMD:R_0603_1608Metric_Pad0.98x0.95mm_HandSolder, symbol Device:R
- R3, R4: value 1k -> 10k
Other:
- note removed: "Figure 2.6 of datasheet Self-powered devices should have this divider from VBUS to protect it from something"

Commit message: Added LEDs to the programmer
Parts:
- added D1, D2: LED, LED_SMD:LED_1206_3216Metric_Pad1.42x1.75mm_HandSolder, symbol Device:LED
- added R6, R7: 500, Resistor_SMD:R_0603_1608Metric_Pad0.98x0.95mm_HandSolder, symbol Device:R
Connections:
- net 3v3: now reaches C3.1, C4.1, R5.2, U7.5 (VIO), U7.6 (VDD)
- net 3v3: now also R6.2, R7.2
- net at U7.13 (~{RXT}/GPIO.1): now also D2.1 (K)
- net at U7.14 (~{TXT}/GPIO.0): now also D1.1 (K)
- new net: D1.2 (A), R7.1
- new net: D2.2 (A), R6.1
- no-connect marks 12 -> 9
